Commit message: revolute type

File: robob/model.urdf (robot description, URDF)
Before this commit: robot robob_platform, 5 links, 4 joints
Links:
- removed link robob_platform__base_link
- removed link robob_platform__left_back_wheel
- removed link robob_platform__left_front_wheel
- removed link robob_platform__right_back_wheel
- removed link robob_platform__right_front_wheel
- added link robob__chassis, mass 0; collision mesh filename=package://robot_description/meshes/robob_platform.dae OR ro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 scale=1.0 1.0 1.0; visual mesh filename=package://robot_description/meshes/robob_platform.dae OR ro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 scale=1.0 1.0 1.0
- added link robob__left_back_wheel, mass 0; collision cylinder length=.02 radius=.03; visual cylinder length=.02 radius=.03
- added link robob__left_front_wheel, mass 0; collision cylinder length=.02 radius=.03; visual cylinder length=.02 radius=.03
- added link robob__right_back_wheel, mass 0; collision cylinder length=.02 radius=.03; visual cylinder length=.02 radius=.03
- added link robob__right_front_wheel, mass 0; collision cylinder length=.02 radius=.03; visual cylinder length=.02 radius=.03
Joints:
- removed joint robob_platform__leftbackwheel_joint
- removed joint robob_platform__leftfrontwheel_joint
- removed joint robob_platform__rightbackwheel_joint
- removed joint robob_platform__rightfrontwheel_joint
- added joint robob__leftbackwheel_joint: type fixed, parent robob__chassis, child robob__left_back_wheel, origin xyz=-0.09  0.09  0.03 rpy=0      1.5707  1.5707, axis 9.00000000e-05   9.00000000e-05   1.00000000e+00, limit lower=0 upper=0 effort=0 velocity=0
- added joint robob__leftfrontwheel_joint: type fixed, parent robob__chassis, child robob__left_front_wheel, origin xyz=0.09  0.09  0.03 rpy=0      1.5707  1.5707, axis 9.00000000e-05   9.00000000e-05   1.00000000e+00, limit lower=0 upper=0 effort=0 velocity=0
- added joint robob__rightbackwheel_joint: type fixed, parent robob__chassis, child robob__right_back_wheel, origin xyz=-0.09 -0.09  0.03 rpy=0      1.5707  1.5707, axis 9.00000000e-05   9.00000000e-05   1.00000000e+00, limit lower=0 upper=0 effort=0 velocity=0
- added joint robob__rightfrontwheel_joint: type fixed, parent robob__chassis, child robob__right_front_wheel, origin xyz=0.09 -0.09  0.03 rpy=0      1.5707  1.5707, axis 9.00000000e-05   9.00000000e-05   1.00000000e+00, limit lower=0 upper=0 effort=0 velocity=0
